File: Romba.kicad_sch (KiCad schematic)
At the start: 7 parts, among them J1 LIDAR UART, J2 Gyro, J3 Buck_5v, J4 Buck_12v, U1 ESP32-DEVKITC-32D, U2 DRV8871DDA, U3 DRV8871DDA

Commit message: PCB
Parts:
- removed U2, U3: DRV8871DDA, Package_SO:Texas_HTSOP-8-1EP_3.9x4.9mm_P1.27mm_EP2.95x4.9mm_Mask2.4x3.1mm_ThermalVias, symbol Driver_Motor:DRV8871DDA
- added U2: TB6612FNG, Package_SO:SSOP-24_5.3x8.2mm_P0.65mm, symbol Driver_Motor:TB6612FNG
Connections:
- new net: U2.1 (AO1), U2.2 (AO1)
- new net: U2.10 (PGND2), U2.9 (PGND2)
- new net: U2.11 (BO1), U2.12 (BO1)
- new net: U2.3 (PGND1), U2.4 (PGND1)
- new net: U2.5 (AO2), U2.6 (AO2)
- new net: U2.7 (BO2), U2.8 (BO2)
Changed lines of the file:
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@@
-	)
-	(symbol
-		(lib_id "Driver_Motor:DRV8871DDA")
-		(at 77.47 66.04 0)
-		(unit 1)
-		(exclude_from_sim no)
-		(in_bom yes)
-		(on_board yes)
-		(dnp no)
-		(fields_autoplaced yes)
-		(property "Reference" "U2"
-			(at 79.6133 53.34 0)
-			(effects
-				(font
-					(size 1.27 1.27)
-				)
-				(justify left)
-			)
-		)
-		(property "Value" "DRV8871DDA"
-			(at 79.6133 55.88 0)
-			(effects
-				(font
-					(size 1.27 1.27)
-				)
-				(justify left)
-			)
-		)
-		(property "Footprint" "Package_SO:Texas_HTSOP-8-1EP_3.9x4.9mm_P1.27mm_EP2.95x4.9mm_Mask2.4x3.1mm_ThermalVias"
-			(at 83.82 67.31 0)
-			(effects
-				(font
-					(size 1.27 1.27)
-				)
-				(hide yes)
-			)
-		)
-		(property "Datasheet" "http://www.ti.com/lit/ds/symlink/drv8871.pdf"
-			(at 83.82 67.31 0)
-			(effects
-				(font
-					(size 1.27 1.27)
-				)
-				(hide yes)
-			)
-		)
-		(property "Description" "Brushed DC Motor Driver, PWM Control, 45V, 3.6A, Current limiting, HTSOP-8"
-			(at 77.47 66.04 0)
-			(effects
-				(font
-					(size 1.27 1.27)
-				)
-				(hide yes)
-			)
-		)
-		(pin "1"
-		)
-		(pin "9"
-		)
-		(pin "6"
-		)
-		(pin "8"
-		)
-		(pin "4"
-		)
-		(pin "7"
-		)
-		(pin "2"
-		)
-		(pin "3"
-		)
-		(pin "5"
-		)
-		(instances
-			(project ""
-				(path "/162ca09a-a45d-4253-9545-f69e74c0a94f"
-					(reference "U2")
-					(unit 1)
-				)
-			)
-		)
 	)
 	(symbol
@@
 	)
 	(symbol
-		(lib_id "Driver_Motor:DRV8871DDA")
-		(at 77.47 95.25 0)
-		(unit 1)
-		(exclude_from_sim no)
-		(in_bom yes)
-		(on_board yes)
-		(dnp no)
-		(fields_autoplaced yes)
-		(property "Reference" "U3"
-			(at 79.6133 82.55 0)
-			(effects
-				(font
-					(size 1.27 1.27)
-				)
-				(justify left)
-			)
-		)
-		(property "Value" "DRV8871DDA"
-			(at 79.6133 85.09 0)
-			(effects
-				(font
-					(size 1.27 1.27)
-				)
-				(justify left)
-			)
-		)
-		(property "Footprint" "Package_SO:Texas_HTSOP-8-1EP_3.9x4.9mm_P1.27mm_EP2.95x4.9mm_Mask2.4x3.1mm_ThermalVias"
-			(at 83.82 96.52 0)
-			(effects
-				(font
-					(size 1.27 1.27)
-				)
-				(hide yes)
-			)
-		)
-		(property "Datasheet" "http://www.ti.com/lit/ds/symlink/drv8871.pdf"
-			(at 83.82 96.52 0)
-			(effects
-				(font
-					(size 1.27 1.27)
-				)
-				(hide yes)
-			)
-		)
-		(property "Description" "Brushed DC Motor Driver, PWM Control, 45V, 3.6A, Current limiting, HTSOP-8"
-			(at 77.47 95.25 0)
-			(effects
-				(font
-					(size 1.27 1.27)
-				)
-				(hide yes)
-			)
-		)
-		(pin "1"
-		)
-		(pin "9"
-		)
-		(pin "6"
-		)
-		(pin "8"
-		)
-		(pin "4"
-		)
-		(pin "7"
-		)
-		(pin "2"
-		)
-		(pin "3"
-		)
-		(pin "5"
-		)
-		(instances
-			(project "Romba"
-				(path "/162ca09a-a45d-4253-9545-f69e74c0a94f"
-					(reference "U3")
-					(unit 1)
-				)
-			)
-		)
-	)
-	(symbol
 		(lib_id "Connector:Conn_01x06_Socket")
 		(at 189.23 96.52 0)
@@
 					(unit 1)
 				)
+			)
+		)
+	)
+	(symbol
+		(lib_id "Driver_Motor:TB6612FNG")
+		(at 49.53 86.36 0)
+		(unit 1)
+		(exclude_from_sim no)
+		(in_bom yes)
+		(on_board yes)
+		(dnp no)
+		(fields_autoplaced yes)
+		(property "Reference" "U2"
+			(at 59.2933 109.22 0)
+			(effects
+				(font
+					(size 1.27 1.27)
+				)
+				(justify left)
+			)
+		)
+		(property "Value" "TB6612FNG"
+			(at 59.2933 111.76 0)
+			(effects
+				(font
+					(size 1.27 1.27)
+				)
+				(justify left)
+			)
+		)
+		(property "Footprint" "Package_SO:SSOP-24_5.3x8.2mm_P0.65mm"
+			(at 82.55 109.22 0)
+			(effects
+				(font
+					(size 1.27 1.27)
+				)
+				(hide yes)
+			)
+		)
+		(property "Datasheet" "https://toshiba.semicon-storage.com/us/product/linear/motordriver/detail.TB6612FNG.html"
+			(at 60.96 71.12 0)
+			(effects
+				(font
+					(size 1.27 1.27)
+				)
+				(hide yes)
+			)
+		)
+		(property "Description" "Driver IC for Dual DC motor, SSOP-24"
+			(at 49.53 86.36 0)
+			(effects
+				(font
+					(size 1.27 1.27)
+				)
+				(hide yes)
+			)
+		)
+		(pin "19"
+		)
+		(pin "18"
+		)
+		(pin "15"
+		)
+		(pin "8"
+		)
+		(pin "17"
+		)
+		(pin "2"
+		)
+		(pin "13"
+		)
+		(pin "16"
+		)
+		(pin "9"
+		)
+		(pin "4"
+		)
+		(pin "1"
+		)
+		(pin "12"
+		)
+		(pin "20"
+		)
+		(pin "23"
+		)
+		(pin "24"
+		)
+		(pin "10"
+		)
+		(pin "11"
+		)
+		(pin "7"
+		)
+		(pin "6"
+		)
+		(pin "3"
+		)
+		(pin "22"
+		)
+		(pin "21"
+		)
+		(pin "14"
+		)
+		(pin "5"
+		)
+		(instances
+			(project ""
+				(path "/162ca09a-a45d-4253-9545-f69e74c0a94f"
+					(reference "U2")
+					(unit 1)
+				)

Commit message: Holy Headache added most footprints
Parts:
- removed J3: Buck_5v, symbol Connector:Conn_01x04_Socket
- removed J4: Buck_12v, symbol Connector:Conn_01x04_Socket
- removed U2: TB6612FNG, Package_SO:SSOP-24_5.3x8.2mm_P0.65mm, symbol Driver_Motor:TB6612FNG
- added 12V_Bulk_Capacitor1: ~1000 microFarads, Capacitor_THT:CP_Radial_D8.0mm_P3.50mm, symbol Device:C
- added 12V_Ceramic_Capacitor1, 5V_Ceramic_Capacitor1, 5V_Ceramic_Capacitor2, 5V_Ceramic_Capacitor3, 5V_Ceramic_Capacitor4, MotorL_HF_Ceramic1, MotorR_HF_Ceramic1: .1 microFarads, Capacitor_SMD:C_0805_2012Metric, symbol Device:C
- added 5V_Bulk_Capacitor1: ~470 microFarads, Capacitor_THT:CP_Radial_D6.3mm_P2.50mm, symbol Device:C
- added FB1, FB2: FerriteBead, Resistor_SMD:R_1206_3216Metric, symbol Device:FerriteBead
- added J3: 5v-Bus, TerminalBlock:TerminalBlock_MaiXu_MX126-5.0-02P_1x02_P5.00mm, symbol Connector:Conn_01x02_Socket
- added J4: 12V-Bus, TerminalBlock:TerminalBlock_MaiXu_MX126-5.0-02P_1x02_P5.00mm, symbol Connector:Conn_01x02_Socket
- added J5: Motor_L, symbol Connector:Conn_01x06_Socket
- added J6: Motor_R, symbol Connector:Conn_01x06_Socket
- added MotorL_Bulk_Ceramic1, MotorR_Bulk_Ceramic1: 47 microFarads, Capacitor_THT:CP_Radial_D5.0mm_P2.00mm, symbol Device:C
- added UMotor_L1, UMotor_R1: DRV8871DDA, Connector_PinHeader_2.54mm:PinHeader_1x04_P2.54mm_Vertical, symbol Driver_Motor:DRV8871DDA
- added UMotor_L2POWER1, UMotor_R2POWER1: DRV8871DDA, TerminalBlock:TerminalBlock_MaiXu_MX126-5.0-02P_1x02_P5.00mm, symbol Driver_Motor:DRV8871DDA
- J1: footprint (none) -> Connector_PinHeader_2.54mm:PinHeader_1x06_P2.54mm_Vertical
- J2: footprint (none) -> Connector_PinHeader_2.54mm:PinHeader_1x08_P2.54mm_Vertical
Connections:
- net Gyro_Gnd is gone; now on net GND: J2.2 (Pin_2)
- net Gyro_Vin is gone; now on net +3.3V: J2.1 (Pin_1)
- net LiDAR_GND is gone; now on net GND: J1.4 (Pin_4)
- net LiDAR_Pwr is gone; now on net +5V: J1.1 (Pin_1)
- net Gyro_SCL\Rx: now also U1.J3-3 (IO22)
- net Gyro_SDA\Tx: now also U1.J3-6 (IO21)
- net LiDAR_RXD/SDA: now also U1.J3-11 (IO17)
- net LiDAR_TXD\SCL: now also U1.J3-12 (IO16)
- net +3.3V: now reaches U1.J2-1 (3V3)
- net +3.3V: now also 5V_Ceramic_Capacitor1.1
- net PWM2_L: now reaches U1.J2-10 (IO26)
- net PWM2_L: now also UMotor_L1.2 (IN2)
- net PWM1_R: now reaches U1.J2-11 (IO27)
- net PWM1_R: now also UMotor_R1.3 (IN1)
- net PWM2_R: now reaches U1.J2-12 (IO14)
- net PWM2_R: now also UMotor_R1.2 (IN2)
- net GND: now reaches U1.J2-14 (GND1)
- net GND: now also U1.J3-1 (GND3), U1.J3-7 (GND2), 12V_Bulk_Capacitor1.2, 12V_Ceramic_Capacitor1.2, 5V_Bulk_Capacitor1.2, 5V_Ceramic_Capacitor1.2, 5V_Ceramic_Capacitor2.2, 5V_Ceramic_Capacitor3.2, 5V_Ceramic_Capacitor4.2, J3.2 (Pin_2), J4.2 (Pin_2), J5.4 (Pin_4), J6.4 (Pin_4), MotorL_Bulk_Ceramic1.2, MotorL_HF_Ceramic1.2, MotorR_Bulk_Ceramic1.2, MotorR_HF_Ceramic1.2, UMotor_L2POWER1.1 (GND), UMotor_L2POWER1.7 (GND), UMotor_L2POWER1.9 (GND), UMotor_R2POWER1.1 (GND), UMotor_R2POWER1.7 (GND), UMotor_R2POWER1.9 (GND)
- net +5V: now reaches U1.J2-19 (EXT_5V)
- net +5V: now also 5V_Ceramic_Capacitor2.1, 5V_Ceramic_Capacitor3.1, FB1.2, J5.3 (Pin_3), J6.3 (Pin_3)
- net EncoderB_L: now reaches U1.J2-5 (IO34)
- net EncoderB_L: now also U1.J2-7 (IO32), J5.1 (Pin_1), J6.1 (Pin_1)
- net EncoderA_R: now reaches U1.J2-6 (IO35)
- net EncoderA_R: now also J6.2 (Pin_2)
- net EncoderA_L: now reaches U1.J2-8 (IO33)
- net EncoderA_L: now also J5.2 (Pin_2)
- net PWM1_L: now reaches U1.J2-9 (IO25)
- net PWM1_L: now also UMotor_L1.3 (IN1)
- new net: UMotor_L1.1 (GND), UMotor_L1.7 (GND), UMotor_L1.9 (GND)
- new net: UMotor_R1.1 (GND), UMotor_R1.7 (GND), UMotor_R1.9 (GND)
- new net +12V: FB2.2, MotorL_Bulk_Ceramic1.1, MotorL_HF_Ceramic1.1, MotorR_Bulk_Ceramic1.1, MotorR_HF_Ceramic1.1, UMotor_L2POWER1.5 (VM), UMotor_R2POWER1.5 (VM)
- new net 12V_Bus: 12V_Bulk_Capacitor1.1, 12V_Ceramic_Capacitor1.1, FB2.1, J4.1 (Pin_1)
- new net 5V_Bus: 5V_Bulk_Capacitor1.1, 5V_Ceramic_Capacitor4.1, FB1.1, J3.1 (Pin_1)
- new net ML+: J5.6 (Pin_6), UMotor_L1.6 (OUT1)
- new net ML-: J5.5 (Pin_5), UMotor_L1.8 (OUT2)
- new net MR+: J6.6 (Pin_6), UMotor_R1.6 (OUT1)
- new net MR-: J6.5 (Pin_5), UMotor_R1.8 (OUT2)
Other:
- moved on the sheet: J1, J2, U1

Commit message: chickenmcnegus
Parts:
- J5, J6: footprint (none) -> Connector_PinHeader_2.54mm:PinHeader_1x06_P2.54mm_Horizontal
- UMotor_L2POWER1, UMotor_R2POWER1: footprint TerminalBlock:TerminalBlock_MaiXu_MX126-5.0-02P_1x02_P5.00mm -> Connector_PinHeader_2.54mm:PinHeader_1x02_P2.54mm_Vertical
Changed lines of the file:
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@@
 			)
 		)
-		(property "Footprint" ""
+		(property "Footprint" "Connector_PinHeader_2.54mm:PinHeader_1x06_P2.54mm_Horizontal"
 			(at 40.64 146.05 0)
 			(effects
@@
 			)
 		)
-		(property "Footprint" "TerminalBlock:TerminalBlock_MaiXu_MX126-5.0-02P_1x02_P5.00mm"
+		(property "Footprint" "Connector_PinHeader_2.54mm:PinHeader_1x02_P2.54mm_Vertical"
 			(at 38.1 102.87 0)
 			(effects
@@
 			)
 		)
-		(property "Footprint" "TerminalBlock:TerminalBlock_MaiXu_MX126-5.0-02P_1x02_P5.00mm"
+		(property "Footprint" "Connector_PinHeader_2.54mm:PinHeader_1x02_P2.54mm_Vertical"
 			(at 74.93 102.87 0)
 			(effects
@@
 			)
 		)
-		(property "Footprint" ""
+		(property "Footprint" "Connector_PinHeader_2.54mm:PinHeader_1x06_P2.54mm_Horizontal"
 			(at 64.77 146.05 0)
 			(effects

Commit message: a bit lost
Parts:
- U1: footprint Amazon ESP32:MODULE_ESP32-DEVKITC-32D -> Battery:BatteryHolder_Keystone_590
Changed lines of the file:
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@@
 			)
 		)
-		(property "Footprint" "Amazon ESP32:MODULE_ESP32-DEVKITC-32D"
+		(property "Footprint" "Battery:BatteryHolder_Keystone_590"
 			(at 132.08 85.09 0)
 			(effects

Commit message: Fixed library issue good to start routing
Parts:
- U1: footprint Battery:BatteryHolder_Keystone_590 -> Amazon ESP32:MODULE_ESP32-DEVKITC-32D
Changed lines of the file:
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@@
 			)
 		)
-		(property "Footprint" "Battery:BatteryHolder_Keystone_590"
+		(property "Footprint" "Amazon ESP32:MODULE_ESP32-DEVKITC-32D"
 			(at 132.08 85.09 0)
 			(effects

Commit message: Finished PCB Routing
Connections:
- net EncoderB_L: no longer J6.1 (Pin_1), U1.J2-5 (IO34)
- net PWM1_L: now also U1.J2-11 (IO27); no longer U1.J2-9 (IO25)
- net PWM1_R: now also U1.J2-9 (IO25); no longer U1.J2-11 (IO27)
- net PWM2_L: now also U1.J2-12 (IO14); no longer U1.J2-10 (IO26)
- net PWM2_R: now also U1.J2-10 (IO26); no longer U1.J2-12 (IO14)
- new net EncoderB_R: J6.1 (Pin_1), U1.J2-5 (IO34)
Changed lines of the file:
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@@
 		)
 	)
-	(label "EncoderB_L"
+	(label "EncoderB_R"
 		(at 111.76 72.39 180)
+		(effects
+			(font
+				(size 1.27 1.27)
+			)
+			(justify right bottom)
+		)
+	)
+	(label "PWM2_L"
+		(at 111.76 90.17 180)
 		(effects
 			(font
@@
 		)
 	)
-	(label "PWM1_R"
-		(at 111.76 87.63 180)
+	(label "PWM2_R"
+		(at 111.76 85.09 180)
 		(effects
 			(font
@@
 		)
 	)
+	(label "PWM1_R"
+		(at 111.76 82.55 180)
+		(effects
+			(font
+				(size 1.27 1.27)
+			)
+			(justify right bottom)
+		)
+	)
 	(label "Gyro_REST"
 		(at 182.88 74.93 180)
@@
 		)
 	)
-	(label "EncoderB_L"
+	(label "EncoderB_R"
 		(at 59.69 140.97 180)
 		(effects
@@
 		)
 	)
-	(label "PWM2_L"
-		(at 111.76 85.09 180)
+	(label "PWM1_L"
+		(at 111.76 87.63 180)
 		(effects
 			(font
@@
 		(effects
 			(font
-				(size 1.27 1.27)
-			)
-			(justify right bottom)
-		)
-	)
-	(label "PWM1_L"
-		(at 111.76 82.55 180)
-		(effects
-			(font
-				(size 1.27 1.27)
-			)
-			(justify right bottom)
-		)
-	)
-	(label "PWM2_R"
-		(at 111.76 90.17 180)
-		(effects
-			(font
